File: MIT PhD/circuits/PD-adder/PD-adder.brd (EAGLE design)
At the start: 100 x 80 mm, 66 parts, among them U1 INA105KP, U2 OP27EZ, U3 OP27EZ, U4 OP27EZ, U5 INA105KP, U6 OP27EZ, U7 REF01EZ, U8 OP27EZ

Commit message: circuit updates
Parts:
- removed C1, C10, C11, C12, C13, C14, C15, C16, C28, C30, C37, C4, C5, C6, C9: 56nF, rcl:C050-030X075
- removed C34, C35, C38, C48: 100uF, rcl:E2,5-6E
- removed C36: 10uF, rcl:C050-030X075
- added C23, C24, C25, C27: 100nF, rcl:C1206
- added C29: (no value), rcl:C1206
- C17, C19, C2, C20, C21, C22, C3, C7, C8: value 100uF -> 100nF; device rcl:E2,5-6E -> rcl:C1206
- C18: value 100uF -> (none); device rcl:E2,5-6E -> rcl:C1206
- C26: value 100uF -> 10uF; device rcl:E2,5-6E -> rcl:C1206
- moved C17 95.6 mm to (90.2, 52.1), turned to 180 degrees
- moved C19 55.7 mm to (29.2, 41.9)
- moved C26 53.4 mm to (58.4, 14.0), turned to 180 degrees
- moved C18 50.4 mm to (74.9, 47.0), turned to 180 degrees
- moved C22 44.5 mm to (90.2, 14.0), turned to 180 degrees
- moved C20 42.3 mm to (59.7, 41.9), turned to 180 degrees
- moved JP5 31.1 mm to (90.2, 67.3)
- moved R9 24.3 mm to (69.8, 31.8), turned to 0 degrees
- moved R19 23.3 mm to (34.3, 6.35), turned to 180 degrees
- moved R2 21.6 mm to (45.7, 48.3), turned to 90 degrees
- moved R4 15.7 mm to (59.7, 72.4)
- moved R5 15.7 mm to (64.8, 72.4)
- moved R8 15.2 mm to (82.5, 58.4)
- moved R3 14.2 mm to (40.6, 72.4), turned to 270 degrees
- moved R15 13.7 mm to (47.0, 30.5)
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Connections:
- net +15V: now also C17.2, C19.2, C20.2, C22.2, C24.1, C25.1, C3.2, C8.2; no longer C11.1, C14.1, C16.1, C18.+, C20.+, C22.+, C3.+, C30.1, C35.+, C37.1, C38.+, C4.1, C48.+, C6.1, C8.+, C9.1
- net -15V: now also C18.1, C2.1, C21.1, C23.1, C27.1, C29.1, C7.1; no longer C1.2, C10.2, C12.2, C13.1, C15.1, C17.-, C19.-, C2.-, C21.-, C26.-, C28.2, C34.-, C5.2, C7.-
- net GND: now also C17.1, C18.2, C19.1, C2.2, C20.1, C21.2, C22.1, C23.2, C24.2, C25.2, C26.1, C27.2, C29.2, C3.1, C7.2, C8.1; no longer C1.1, C10.1, C11.2, C12.1, C13.2, C14.2, C15.2, C16.2, C17.+, C18.-, C19.+, C2.+, C20.-, C21.+, C22.-, C26.+, C28.1, C3.-, C30.2, C34.+, C35.-, C36.2, C37.2, C38.-, C4.2, C48.-, C5.1, C6.2, C7.+, C8.-, C9.2
- net N$21: now also C26.2; no longer C36.1
Routing:
- net GND: track 488.7 -> 402.4 mm, vias 1 -> 0
- net N$12: track 121.7 -> 63.8 mm, vias 0 -> 1
- net N$21: track 70.8 -> 32.1 mm
- net N$8: track 76.4 -> 47.8 mm, vias 0 -> 1
- net -15V: track 258.0 -> 230.8 mm
- net N$6: track 3.18 -> 26.0 mm
- net N$15: track 53.6 -> 31.2 mm
- net N$7: track 38.5 -> 16.5 mm
- net N$9: track 29.8 -> 10.3 mm
- net +15V: track 245.0 -> 229.6 mm
- net N$3: track 11.5 -> 21.9 mm
- net N$2: track 7.50 -> 17.7 mm
- net V_OUT: track 14.1 -> 21.8 mm
- net VOUT: track 7.94 -> 15.4 mm
- net N$13: track 12.1 -> 5.18 mm
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
Commit message: circuits
Parts:
- added C1, C10, C11, C12, C4, C5, C6, C9: (no value), discrete:ES-2,5
- added C13, C14, C15, C16, C28, C30, C31, C32: 100 nf, rcl:C0805
- added IC1: ADG221KN, linear:DIL16
- added IC4: (no value), v-reg:79XXL
- added IC5: (no value), v-reg:78XXL
- added IC6, IC7: LF347N, linear:DIL14
- added IC8: ADG222KN, linear:DIL16
- added POWER_IN: (no value), con-amp:10X03MTA
- C17, C18, C19, C2, C20, C21, C22, C23, C24, C25, C26, C27, C29, C3, C7, C8: device rcl:C1206 -> rcl:C1206@1
Connections:
- new net +18V: C1.1, C5.1, IC5.IN, POWER_IN.3
- new net -18V: C4.2, C6.2, IC4.IN, POWER_IN.1
- net +15V: now also C10.1, C13.1, C15.1, C31.1, C32.1, C9.1, IC1.13, IC5.OUT, IC6.4, IC7.4, IC8.13
- net -15V: now also C11.2, C12.2, C14.2, C16.2, C28.2, C30.2, IC1.4, IC4.OUT, IC6.11, IC7.11, IC8.4
- net GND: now also C1.2, C10.2, C11.1, C12.1, C13.2, C14.1, C15.2, C16.1, C28.1, C30.1, C31.2, C32.2, C4.1, C5.2, C6.1, C9.2, IC1.5, IC4.GND, IC5.GND, IC8.5, POWER_IN.2

Commit message: circuits
Parts:
- C1, C10, C11, C12, C4, C5, C6, C9: value (none) -> 1uF
- C13, C14, C15, C16, C28, C30, C31, C32: value 100 nf -> 100nF
- C29: value (none) -> 100nF
- moved C15 106.1 mm to (81.3, 12.7)
- moved C13 97.0 mm to (96.5, 19.1), turned to 90 degrees
- moved C16 90.3 mm to (67.3, 11.4), turned to 90 degrees
- moved C30 88.6 mm to (66.0, 20.3), turned to 90 degrees
- moved C14 84.2 mm to (83.8, 19.1), turned to 90 degrees
- moved C11 81.3 mm to (27.9, 25.4), turned to 270 degrees
- moved C12 81.0 mm to (31.8, 25.4), turned to 270 degrees
- moved C32 80.8 mm to (52.1, 21.6), turned to 180 degrees
- moved C28 80.1 mm to (52.1, 14.0), turned to 180 degrees
- moved IC7 79.8 mm to (59.7, 21.6), turned to 270 degrees
- moved C10 78.8 mm to (6.35, 25.4), turned to 90 degrees
- moved C9 73.8 mm to (10.2, 25.4), turned to 90 degrees
- moved IC8 73.3 mm to (73.7, 11.4), turned to 270 degrees
- moved C31 72.5 mm to (36.8, 14.0), turned to 180 degrees
- moved IC1 60.2 mm to (90.2, 19.1), turned to 270 degrees
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Connections:
- new net N$1: C13.2, C14.1, IC1.5
- net GND: no longer C13.2, C14.1, IC1.5
Routing:
- net GND: track 402.4 -> 541.2 mm, vias 0 -> 1
- net +15V: track 229.6 -> 323.1 mm
- net -15V: track 230.8 -> 307.8 mm
- net -18V: track 0.00 -> 21.5 mm
- net +18V: track 0.00 -> 19.1 mm
- net N$20: track 20.1 -> 38.4 mm, vias 1 -> 0
- net N$1: track 0.00 -> 16.4 mm
- net N$8: track 47.8 -> 34.8 mm
- net N$21: track 32.1 -> 22.2 mm, vias 0 -> 1
- net N$14: track 14.8 -> 5.40 mm, vias 0 -> 1
- net N$5: track 35.4 -> 28.2 mm
- net N$2: track 17.7 -> 11.0 mm
- net N$9: track 10.3 -> 3.91 mm
- net N$17: track 56.2 -> 62.3 mm
- net N$10: track 50.2 -> 46.4 mm
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