File: MIT PhD/circuits/PD-adder/PD-adder.sch (EAGLE design)
At the start: 61 parts, among them U1 INA105KP, U2 OP27EZ, U3 OP27EZ, U4 OP27EZ, U5 INA105KP, U6 OP27EZ, U7 REF01EZ, U8 OP27EZ

Commit message: circuits
Parts:
- added JP1, JP2, JP3, JP4, JP5: (no value), pinhead:PINHD-1X1
Connections:
- removed net VCC: C13.1, C14.1, C15.1, C17.-, C18.+, C19.-, C20.+, C37.1, C38.+, C9.1, U6.V+, U6.V-, U7.VIN, U8.V+, U8.V-
- new net -15V: C1.2, C10.2, C12.2, C13.1, C15.1, C17.-, C19.-, C2.-, C21.-, C26.-, C28.2, C34.-, C5.2, C7.-, U1.V-, U2.V-, U3.V-, U4.V-, U5.V-, U6.V-, U8.V-
- net +15V: now also C14.1, C18.+, C20.+, C37.1, C38.+, C9.1, U6.V+, U7.VIN, U8.V+; no longer C1.2, C10.2, C12.2, C2.-, C21.-, C26.-, C28.2, C34.-, C5.2, C7.-, U1.V-, U2.V-, U3.V-, U4.V-, U5.V-
- net N$1: now also R1.1
- net N$12: now also D1.C
- net VHI-IN+: now also JP1.1
- net VHI-IN-: now also JP2.1
- net VLO-IN+: now also JP3.1
- net VLO-IN-: now also JP4.1
- net V_OUT: now also JP5.1
Other:
- moved on the sheet: R17

Commit message: circuit updates
Parts:
- removed C1, C10, C11, C12, C13, C14, C15, C16, C28, C30, C37, C4, C5, C6, C9: 56nF, rcl:C-EU050-030X075
- removed C34, C35, C38, C48: 100uF, rcl:CPOL-USE2,5-6E
- removed C36: 10uF, rcl:C-EU050-030X075
- added C23, C24, C25, C27: 100nF, rcl:C-EUC1206
- added C29: (no value), rcl:C-EUC1206
- C17, C19, C2, C20, C21, C22, C3, C7, C8: value 100uF -> 100nF; device rcl:CPOL-USE2,5-6E -> rcl:C-EUC1206
- C18: value 100uF -> (none); device rcl:CPOL-USE2,5-6E -> rcl:C-EUC1206
- C26: value 100uF -> 10uF; device rcl:CPOL-USE2,5-6E -> rcl:C-EUC1206
Connections:
- net +15V: now also C17.2, C19.2, C20.2, C22.2, C24.1, C25.1, C3.2, C8.2; no longer C11.1, C14.1, C16.1, C18.+, C20.+, C22.+, C3.+, C30.1, C35.+, C37.1, C38.+, C4.1, C48.+, C6.1, C8.+, C9.1
- net -15V: now also C18.1, C2.1, C21.1, C23.1, C27.1, C29.1, C7.1; no longer C1.2, C10.2, C12.2, C13.1, C15.1, C17.-, C19.-, C2.-, C21.-, C26.-, C28.2, C34.-, C5.2, C7.-
- net GND: now also C17.1, C18.2, C19.1, C2.2, C20.1, C21.2, C22.1, C23.2, C24.2, C25.2, C26.1, C27.2, C29.2, C3.1, C7.2, C8.1; no longer C1.1, C10.1, C11.2, C12.1, C13.2, C14.2, C15.2, C16.2, C17.+, C18.-, C19.+, C2.+, C20.-, C21.+, C22.-, C26.+, C28.1, C3.-, C30.2, C34.+, C35.-, C36.2, C37.2, C38.-, C4.2, C48.-, C5.1, C6.2, C7.+, C8.-, C9.2
- net N$21: now also C26.2; no longer C36.1
Other:
- moved on the sheet: R1

Commit message: circuits
Parts:
- added C1, C10, C11, C12, C4, C5, C6, C9: (no value), discrete:ELC-2,5
- added C13, C14, C15, C16, C28, C30, C31, C32: 100 nf, rcl:C-USC0805
- added IC1: ADG221KN, linear:ADG221KN
- added IC4: (no value), v-reg:79XXL
- added IC5: (no value), v-reg:78XXL
- added IC6, IC7: LF347N, linear:LF347N
- added IC8: ADG222KN, linear:ADG222KN
- added POWER_IN: (no value), con-amp:MTA03-100
Connections:
- new net +18V: C1.1, C5.1, IC5.IN, POWER_IN.3
- new net -18V: C4.2, C6.2, IC4.IN, POWER_IN.1
- net +15V: now also C10.1, C13.1, C15.1, C31.1, C32.1, C9.1, IC1P.V+, IC5.OUT, IC6P.V+, IC7P.V+, IC8P.V+
- net -15V: now also C11.2, C12.2, C14.2, C16.2, C28.2, C30.2, IC1P.V-, IC4.OUT, IC6P.V-, IC7P.V-, IC8P.V-
- net GND: now also C1.2, C10.2, C11.1, C12.1, C13.2, C14.1, C15.2, C16.1, C28.1, C30.1, C31.2, C32.2, C4.1, C5.2, C6.1, C9.2, IC1P.GND, IC4.GND, IC5.GND, IC8P.GND, POWER_IN.2

Commit message: circuits
Parts:
- C1, C10, C11, C12, C4, C5, C6, C9: value (none) -> 1uF
- C13, C14, C15, C16, C28, C30, C31, C32: value 100 nf -> 100nF
- C29: value (none) -> 100nF
Connections:
- new net N$1: C13.2, C14.1, IC1P.GND
- net GND: no longer C13.2, C14.1, IC1P.GND
Other:
- moved on the sheet: C1, C10, C11, C12, C13, C14, C15, C16, C28, C30, C31, C32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
